File: botonera.sch (KiCad schematic (older format))
At the start: 17 parts, among them J1 VCC, J2 RST, J3 BUTTON1, J4 BUTTON2, J5 LIGHT1, J6 LIGHT2, K1 SUNHOLD_RAS_Form_C, K2 SUNHOLD_RAS_Form_C, K3 SUNHOLD_RAS_Form_C, M1 MOUNTING-HOLE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

Commit message: esquematico y pcb generado
Parts:
- removed D1: D_PSH_PLY1, Diodes_ThroughHole:Diode_DO-35_SOD27_Horizontal_RM10, symbol D
- removed D2: D_PSH_PLY2, Diodes_ThroughHole:Diode_DO-35_SOD27_Horizontal_RM10, symbol D
- removed D3: D_LED_PLY1, Diodes_ThroughHole:Diode_DO-35_SOD27_Horizontal_RM10, symbol D
- removed D4: D_LED_PLY2, Diodes_ThroughHole:Diode_DO-35_SOD27_Horizontal_RM10, symbol D
- removed J1: VCC, Terminal_Blocks:TerminalBlock_Pheonix_MKDS1.5-2pol, symbol Screw_Terminal_1x02
- removed J2: RST, Terminal_Blocks:TerminalBlock_Pheonix_MKDS1.5-2pol, symbol Screw_Terminal_1x02
- removed J3: BUTTON1, Terminal_Blocks:TerminalBlock_Pheonix_MKDS1.5-2pol, symbol Screw_Terminal_1x02
- removed J4: BUTTON2, Terminal_Blocks:TerminalBlock_Pheonix_MKDS1.5-2pol, symbol Screw_Terminal_1x02
- removed J5: LIGHT1, Terminal_Blocks:TerminalBlock_Pheonix_MKDS1.5-2pol, symbol Screw_Terminal_1x02
- removed J6: LIGHT2, Terminal_Blocks:TerminalBlock_Pheonix_MKDS1.5-2pol, symbol Screw_Terminal_1x02
- removed K1, K2, K3: SUNHOLD_RAS_Form_C, edseen_relay:Relay_SUNHOLD_RAS_Series_Form_C, symbol SUNHOLD_RAS_Form_C
- removed M1, M2, M3, M4: MOUNTING-HOLE, Connect:1pin, symbol MOUNTING-HOLE
- added D1: D_PSH_PLY1, Diode_THT:D_DO-41_SOD81_P10.16mm_Horizontal, symbol Diode:1N4004
- added D2: D_PSH_PLY2, Diode_THT:D_DO-41_SOD81_P10.16mm_Horizontal, symbol Diode:1N4004
- added D3: D_LED_PLY1, Diode_THT:D_DO-41_SOD81_P10.16mm_Horizontal, symbol Diode:1N4004
- added D4: D_LED_PLY2, Diode_THT:D_DO-41_SOD81_P10.16mm_Horizontal, symbol Diode:1N4004
- added J1: VCC, TerminalBlock_TE-Connectivity:TerminalBlock_TE_282834-2_1x02_P2.54mm_Horizontal, symbol Connector:Screw_Terminal_01x02
- added J2: RST, TerminalBlock_TE-Connectivity:TerminalBlock_TE_282834-2_1x02_P2.54mm_Horizontal, symbol Connector:Screw_Terminal_01x02
- added J3: BUTTON1, TerminalBlock_TE-Connectivity:TerminalBlock_TE_282834-2_1x02_P2.54mm_Horizontal, symbol Connector:Screw_Terminal_01x02
- added J4: BUTTON2, TerminalBlock_TE-Connectivity:TerminalBlock_TE_282834-2_1x02_P2.54mm_Horizontal, symbol Connector:Screw_Terminal_01x02
- added J5: LIGHT1, TerminalBlock_TE-Connectivity:TerminalBlock_TE_282834-2_1x02_P2.54mm_Horizontal, symbol Connector:Screw_Terminal_01x02
- added J6: LIGHT2, TerminalBlock_TE-Connectivity:TerminalBlock_TE_282834-2_1x02_P2.54mm_Horizontal, symbol Connector:Screw_Terminal_01x02
- added K1: MAIN, edseen_relay:Relay_SUNHOLD_RAS_Series_Form_C, symbol edseen_relay:SUNHOLD_RAS_Form_C
- added K2: PLY1, edseen_relay:Relay_SUNHOLD_RAS_Series_Form_C, symbol edseen_relay:SUNHOLD_RAS_Form_C
- added K3: PLY2, edseen_relay:Relay_SUNHOLD_RAS_Series_Form_C, symbol edseen_relay:SUNHOLD_RAS_Form_C
Connections:
- net BUTTON1_1: now also D1.1 (K), J3.1 (Pin_1)
- net BUTTON1_2: now also D3.2 (A), J3.2 (Pin_2), J5.1 (Pin_1), K2.1 (Coil), K2.5 (NO)
- net BUTTON2_1: now also D2.1 (K), J4.2 (Pin_2)
- net BUTTON2_2: now also D4.2 (A), J4.1 (Pin_1), J6.2 (Pin_2), K3.1 (Coil), K3.5 (NO)
- net GND: now also D3.1 (K), D4.1 (K), J1.1 (Pin_1), K1.1 (Coil), K1.2 (Coil), K1.5 (NO)
- net Vcc2: now also J2.2 (Pin_2), K1.3 (Common), K2.3 (Common), K3.3 (Common)
- new net: J5.2 (Pin_2), J6.1 (Pin_1), K2.2 (Coil), K3.2 (Coil)
- new net: D1.2 (A), D2.2 (A), K1.4 (NC)
- new net +5V: J1.2 (Pin_2), J2.1 (Pin_1)
- no-connect marks 0 -> 2
